Commit message: gazebo lesson

File: my_robot_description/urdf/common_properties.xacro (robot description, xacro)
@@ -10,3 +10,33 @@
     <color rgba="0.5 0.5 0.5 1" />
   </material>
+  <xacro:macro name="box_inertial" params="mass size_x size_y size_z o_xyz o_rpy">
+    <inertial>
+      <mass value="${mass}" />
+      <inertia
+        ixx="${mass / 12.0 * (size_y * size_y + size_z * size_z)}" ixy="0" ixz="0"
+        iyy="${mass / 12.0 * (size_z * size_z + size_x * size_x)}" iyz="0"
+        izz="${mass / 12.0 * (size_x * size_x + size_y * size_y)}" />
+      <origin xyz="${o_xyz}" rpy="${o_rpy}" />
+    </inertial>
+  </xacro:macro>
+  <xacro:macro name="cylinder_inertial" params="mass radius length o_xyz o_rpy">
+    <inertial>
+      <mass value="${mass}" />
+      <inertia
+        ixx="${mass / 12.0 * (3.0 * radius * radius + length * length)}" ixy="0" ixz="0"
+        iyy="${mass / 12.0 * (3.0 * radius * radius + length * length)}" iyz="0"
+        izz="${mass / 2.0 * radius * radius}" />
+      <origin xyz="${o_xyz}" rpy="${o_rpy}" />
+    </inertial>
+  </xacro:macro>
+  <xacro:macro name="sphere_inertial" params="mass radius o_xyz o_rpy">
+    <inertial>
+      <mass value="${mass}" />
+      <inertia
+        ixx="${2.0 * mass / 5.0 * radius * radius}" ixy="0" ixz="0"
+        iyy="${2.0 * mass / 5.0 * radius * radius}" iyz="0"
+        izz="${2.0 * mass / 5.0 * radius * radius}" />
+      <origin xyz="${o_xyz}" rpy="${o_rpy}" />
+    </inertial>
+  </xacro:macro>
 </robot>

File: my_robot_description/urdf/mobile_base.xacro (robot description, xacro)
@@ -6,4 +6,7 @@
   <xacro:property name="wheel_radius" value="0.1" />
   <xacro:property name="wheel_width" value="0.05" />
+  <xacro:property name="base_mass" value="5.0" />
+  <xacro:property name="wheel_mass" value="1.0" />
+  <xacro:property name="caster_mass" value="0.5" />
   <link name="base_footprint" />
   <link name="base_link">
@@ -15,4 +18,13 @@
       <material name="blue" />
     </visual>
+    <collision>
+      <geometry>
+        <box size="${base_length} ${base_width} ${base_height}" />
+      </geometry>
+      <origin xyz="0 0 ${base_height / 2.0}" rpy="0 0 0" />
+    </collision>
+    <xacro:box_inertial mass="${base_mass}"
+      size_x="${base_length}" size_y="${base_width}" size_z="${base_height}"
+      o_xyz="0 0 ${base_height / 2.0}" o_rpy="0 0 0" />
   </link>
   <xacro:macro name="wheel_link" params="prefix">
@@ -25,4 +37,13 @@
         <material name="gray" />
       </visual>
+      <collision>
+        <geometry>
+          <sphere radius="${wheel_radius}" />
+        </geometry>
+        <origin xyz="0 0 0" rpy="0 0 0" />
+      </collision>
+      <xacro:cylinder_inertial mass="${wheel_mass}"
+        radius="${wheel_radius}" length="${wheel_width}"
+        o_xyz="0 0 0" o_rpy="${pi / 2.0} 0 0" />
     </link>
   </xacro:macro>
@@ -37,4 +58,13 @@
       <material name="gray" />
     </visual>
+    <collision>
+      <geometry>
+        <sphere radius="${wheel_radius / 2.0}" />
+      </geometry>
+      <origin xyz="0 0 0" rpy="0 0 0" />
+    </collision>
+    <xacro:sphere_inertial mass="${caster_mass}"
+      radius="${wheel_radius / 2.0}"
+      o_xyz="0 0 0" o_rpy="0 0 0" />
   </link>
   <joint name="base_joint" type="fixed">
@@ -43,5 +73,5 @@
     <origin xyz="0 0 ${wheel_radius}" rpy="0 0 0" />
   </joint>
-  <joint name="base_rigth_wheel_joint" type="continuous">
+  <joint name="base_right_wheel_joint" type="continuous">
     <parent link="base_link" />
     <child link="right_wheel_link" />
@@ -55,5 +85,5 @@
     <axis xyz="0 1 0" />
   </joint>
-  <joint name="base=caster_wheel_joint" type="fixed">
+  <joint name="base_caster_wheel_joint" type="fixed">
     <parent link="base_link" />
     <child link="caster_wheel_link" />

File: my_robot_description/urdf/my_robot.urdf.xacro (robot description, xacro)
@@ -3,3 +3,4 @@
   <xacro:include filename="common_properties.xacro" />
   <xacro:include filename="mobile_base.xacro" />
+  <xacro:include filename="mobile_base_gazebo.xacro" />
 </robot>

Commit message: final project

File: my_robot_description/urdf/common_properties.xacro (robot description, xacro)
@@ -1,4 +1,7 @@
 <?xml version="1.0" encoding="UTF-8"?>
 <robot xmlns:xacro="http://www.ros.org/wiki/xacro">
+  <material name="red">
+    <color rgba="0.5 0 0 1" />
+  </material>
   <material name="green">
     <color rgba="0 0.5 0 1" />
@@ -9,4 +12,10 @@
   <material name="gray">
     <color rgba="0.5 0.5 0.5 1" />
+  </material>
+  <material name="orange">
+    <color rgba="1 0.5 0 1" />
+  </material>
+  <material name="yellow">
+    <color rgba="1 1 0 1" />
   </material>
   <xacro:macro name="box_inertial" params="mass size_x size_y size_z o_xyz o_rpy">

File: my_robot_description/urdf/mobile_base.xacro (robot description, xacro)
@@ -15,5 +15,5 @@
         <box size="${base_length} ${base_width} ${base_height}" />
       </geometry>
-      <origin xyz="0 0 ${base_height / 2.0}" rpy="0 0 0" />
+      <origin xyz="0 0 ${base_height / 2}" rpy="0 0 0" />
       <material name="blue" />
     </visual>
@@ -22,9 +22,9 @@
         <box size="${base_length} ${base_width} ${base_height}" />
       </geometry>
-      <origin xyz="0 0 ${base_height / 2.0}" rpy="0 0 0" />
+      <origin xyz="0 0 ${base_height / 2}" rpy="0 0 0" />
     </collision>
     <xacro:box_inertial mass="${base_mass}"
       size_x="${base_length}" size_y="${base_width}" size_z="${base_height}"
-      o_xyz="0 0 ${base_height / 2.0}" o_rpy="0 0 0" />
+      o_xyz="0 0 ${base_height / 2}" o_rpy="0 0 0" />
   </link>
   <xacro:macro name="wheel_link" params="prefix">
@@ -34,5 +34,5 @@
           <cylinder radius="${wheel_radius}" length="${wheel_width}" />
         </geometry>
-        <origin xyz="0 0 0" rpy="${pi / 2.0} 0 0" />
+        <origin xyz="0 0 0" rpy="${pi / 2} 0 0" />
         <material name="gray" />
       </visual>
@@ -45,5 +45,5 @@
       <xacro:cylinder_inertial mass="${wheel_mass}"
         radius="${wheel_radius}" length="${wheel_width}"
-        o_xyz="0 0 0" o_rpy="${pi / 2.0} 0 0" />
+        o_xyz="0 0 0" o_rpy="${pi / 2} 0 0" />
     </link>
   </xacro:macro>
@@ -53,5 +53,5 @@
     <visual>
       <geometry>
-        <sphere radius="${wheel_radius / 2.0}" />
+        <sphere radius="${wheel_radius / 2}" />
       </geometry>
       <origin xyz="0 0 0" rpy="0 0 0" />
@@ -60,10 +60,10 @@
     <collision>
       <geometry>
-        <sphere radius="${wheel_radius / 2.0}" />
+        <sphere radius="${wheel_radius / 2}" />
       </geometry>
       <origin xyz="0 0 0" rpy="0 0 0" />
     </collision>
     <xacro:sphere_inertial mass="${caster_mass}"
-      radius="${wheel_radius / 2.0}"
+      radius="${wheel_radius / 2}"
       o_xyz="0 0 0" o_rpy="0 0 0" />
   </link>
@@ -76,5 +76,5 @@
     <parent link="base_link" />
     <child link="right_wheel_link" />
-    <origin xyz="${-base_length / 4} ${-(base_width + wheel_width) / 2.0} 0" rpy="0 0 0" />
+    <origin xyz="${-base_length / 4} ${-(base_width + wheel_width) / 2} 0" rpy="0 0 0" />
     <axis xyz="0 1 0" />
   </joint>
@@ -82,5 +82,5 @@
     <parent link="base_link" />
     <child link="left_wheel_link" />
-    <origin xyz="${-base_length / 4} ${(base_width + wheel_width) / 2.0}  0" rpy="0 0 0" />
+    <origin xyz="${-base_length / 4} ${(base_width + wheel_width) / 2}  0" rpy="0 0 0" />
     <axis xyz="0 1 0" />
   </joint>
@@ -88,5 +88,5 @@
     <parent link="base_link" />
     <child link="caster_wheel_link" />
-    <origin xyz="${base_length / 3} 0 ${-wheel_radius / 2.0}" rpy="0 0 0" />
+    <origin xyz="${base_length / 3} 0 ${-wheel_radius / 2}" rpy="0 0 0" />
   </joint>
 </robot>

File: my_robot_description/urdf/my_robot.urdf.xacro (robot description, xacro)
@@ -4,4 +4,11 @@
   <xacro:include filename="mobile_base.xacro" />
   <xacro:include filename="mobile_base_gazebo.xacro" />
+  <xacro:include filename="arm.xacro" />
+  <xacro:include filename="arm_gazebo.xacro" />
   <xacro:include filename="camera.xacro" />
+  <joint name="mobile_base_arm_joint" type="fixed">
+    <parent link="base_link" />
+    <child link="arm_base_link" />
+    <origin xyz="${base_length / 4} 0 ${base_height}" rpy="0 0 0" />
+  </joint>
 </robot>
