Commit message: separate materials and interial files, separate origin on intertial macros

File: my_robot_description/urdf/arm.xacro (robot description, xacro)
@@ -25,7 +25,8 @@
       <origin xyz="0 0 ${arm_base_height / 2}" rpy="0 0 0" />
     </collision>
-    <xacro:box_inertial mass="${arm_base_mass}"
-      size_x="${arm_base_length}" size_y="${arm_base_width}" size_z="${arm_base_height}"
-      o_xyz="0 0 ${arm_base_height / 2}" o_rpy="0 0 0" />
+    <xacro:inertial_box mass="${arm_base_mass}"
+      x="${arm_base_length}" y="${arm_base_width}" z="${arm_base_height}">
+      <origin xyz="0 0 ${arm_base_height / 2}" rpy="0 0 0" />
+    </xacro:inertial_box>
   </link>
   <link name="forearm_link">
@@ -43,7 +44,8 @@
       <origin xyz="0 0 ${forearm_length / 2}" rpy="0 0 0" />
     </collision>
-    <xacro:cylinder_inertial mass="${forearm_mass}"
-      radius="${forearm_radius}" length="${forearm_length}"
-      o_xyz="0 0 ${forearm_length / 2}" o_rpy="0 0 0" />
+    <xacro:inertial_cylinder mass="${forearm_mass}"
+      radius="${forearm_radius}" length="${forearm_length}">
+      <origin xyz="0 0 ${forearm_length / 2}" rpy="0 0 0" />
+    </xacro:inertial_cylinder>
   </link>
   <link name="hand_link">
@@ -61,7 +63,8 @@
       <origin xyz="0 0 ${hand_length / 2}" rpy="0 0 0" />
     </collision>
-    <xacro:cylinder_inertial mass="${hand_mass}"
-      radius="${hand_radius}" length="${hand_length}"
-      o_xyz="0 0 ${hand_length / 2}" o_rpy="0 0 0" />
+    <xacro:inertial_cylinder mass="${hand_mass}"
+      radius="${hand_radius}" length="${hand_length}">
+      <origin xyz="0 0 ${hand_length / 2}" rpy="0 0 0" />
+    </xacro:inertial_cylinder>
   </link>
   <joint name="arm_base_forearm_joint" type="revolute">

File: my_robot_description/urdf/camera.xacro (robot description, xacro)
@@ -17,7 +17,8 @@
       </geometry>
     </collision>
-    <xacro:box_inertial mass="${camera_mass}"
-      size_x="${camera_length}" size_y="${camera_width}" size_z="${camera_height}"
-      o_xyz="0 0 0" o_rpy="0 0 0" />
+    <xacro:inertial_box mass="${camera_mass}"
+      x="${camera_length}" y="${camera_width}" z="${camera_height}">
+      <origin xyz="0 0 0" rpy="0 0 0" />
+    </xacro:inertial_box>
   </link>
   <link name="camera_link_optical" />

File: my_robot_description/urdf/mobile_base.xacro (robot description, xacro)
@@ -24,7 +24,8 @@
       <origin xyz="0 0 ${base_height / 2}" rpy="0 0 0" />
     </collision>
-    <xacro:box_inertial mass="${base_mass}"
-      size_x="${base_length}" size_y="${base_width}" size_z="${base_height}"
-      o_xyz="0 0 ${base_height / 2}" o_rpy="0 0 0" />
+    <xacro:inertial_box mass="${base_mass}"
+      x="${base_length}" y="${base_width}" z="${base_height}">
+      <origin xyz="0 0 ${base_height / 2}" rpy="0 0 0" />
+    </xacro:inertial_box>
   </link>
   <xacro:macro name="wheel_link" params="prefix">
@@ -43,7 +44,8 @@
         <origin xyz="0 0 0" rpy="0 0 0" />
       </collision>
-      <xacro:cylinder_inertial mass="${wheel_mass}"
-        radius="${wheel_radius}" length="${wheel_width}"
-        o_xyz="0 0 0" o_rpy="${pi / 2} 0 0" />
+      <xacro:inertial_cylinder mass="${wheel_mass}"
+        radius="${wheel_radius}" length="${wheel_width}">
+        <origin xyz="0 0 0" rpy="${pi / 2} 0 0" />
+      </xacro:inertial_cylinder>
     </link>
   </xacro:macro>
@@ -64,7 +66,8 @@
       <origin xyz="0 0 0" rpy="0 0 0" />
     </collision>
-    <xacro:sphere_inertial mass="${caster_mass}"
-      radius="${wheel_radius / 2}"
-      o_xyz="0 0 0" o_rpy="0 0 0" />
+    <xacro:inertial_sphere mass="${caster_mass}"
+      radius="${wheel_radius / 2}">
+      <origin xyz="0 0 0" rpy="0 0 0" />
+    </xacro:inertial_sphere>
   </link>
   <joint name="base_joint" type="fixed">

File: my_robot_description/urdf/my_robot.urdf.xacro (robot description, xacro)
@@ -1,5 +1,6 @@
 <?xml version="1.0" encoding="UTF-8"?>
 <robot name="my_robot" xmlns:xacro="http://www.ros.org/wiki/xacro">
-  <xacro:include filename="common_properties.xacro" />
+  <xacro:include filename="materials.xacro" />
+  <xacro:include filename="inertial_macros.xacro" />
   <xacro:include filename="mobile_base.xacro" />
   <xacro:include filename="mobile_base_gazebo.xacro" />

File: my_robot_description/urdf/standalone_arm.urdf.xacro (robot description, xacro)
@@ -1,5 +1,6 @@
 <?xml version="1.0" encoding="UTF-8"?>
 <robot name="my_robot" xmlns:xacro="http://www.ros.org/wiki/xacro">
-  <xacro:include filename="common_properties.xacro" />
+  <xacro:include filename="materials.xacro" />
+  <xacro:include filename="inertial_macros.xacro" />
   <xacro:include filename="arm.xacro" />
   <xacro:include filename="arm_gazebo.xacro" />
